Commit message: Add factory fleet dashboard, traffic coordination, cargo and Sketchfab assets

File: src/factory_bot/urdf/fleet_bot.gazebo.xacro (robot description, xacro)
@@ -32,4 +32,6 @@
       <visualize>false</visualize>
       <lidar>
+        <!-- Ordinary geometry plus the forklift's lidar-only outer bounding box. -->
+        <visibility_mask>2415919103</visibility_mask>
         <scan>
           <horizontal>
@@ -53,4 +55,39 @@
     </sensor>
   </gazebo>
+  <!-- 91 low front rays: body-height obstacle detection, not a SLAM input. -->
+  <gazebo reference="obstacle_laser_link">
+    <sensor name="obstacle_lidar_${ns}" type="gpu_lidar">
+      <topic>${ns}/obstacle_scan</topic>
+      <gz_frame_id>${ns}/obstacle_laser_link</gz_frame_id>
+      <update_rate>10</update_rate><always_on>true</always_on><visualize>false</visualize>
+      <lidar>
+        <visibility_mask>2415919103</visibility_mask>
+        <scan><horizontal><samples>91</samples><resolution>1</resolution>
+          <min_angle>-0.7853981633974483</min_angle><max_angle>0.7853981633974483</max_angle>
+        </horizontal></scan>
+        <range><min>0.02</min><max>4.0</max><resolution>0.01</resolution></range>
+        <noise><type>gaussian</type><mean>0.0</mean><stddev>0.005</stddev></noise>
+      </lidar>
+    </sensor>
+  </gazebo>
+  <!-- First-person RGB camera. Sensor forward = +X; ROS optical frame = +Z forward. -->
+  <xacro:if value="$(arg cameras)">
+    <gazebo reference="camera_link">
+      <sensor name="front_camera_${ns}" type="camera">
+        <topic>${ns}/camera/image_raw</topic>
+        <gz_frame_id>${ns}/camera_optical_frame</gz_frame_id>
+        <update_rate>$(arg camera_rate)</update_rate>
+        <always_on>true</always_on><visualize>false</visualize>
+        <camera>
+          <!-- Exclude lidar-only collision envelopes from RGB images. -->
+          <visibility_mask>268435455</visibility_mask>
+          <camera_info_topic>${ns}/camera/camera_info</camera_info_topic>
+          <horizontal_fov>1.3962634</horizontal_fov>
+          <image><width>$(arg camera_width)</width><height>$(arg camera_height)</height><format>R8G8B8</format><anti_aliasing>2</anti_aliasing></image>
+          <clip><near>0.025</near><far>24.0</far></clip>
+        </camera>
+      </sensor>
+    </gazebo>
+  </xacro:if>
   <!-- IMU: measures turning and acceleration, 100 times per second -->
   <gazebo reference="imu_link">

File: src/factory_bot/urdf/fleet_bot.urdf.xacro (robot description, xacro)
@@ -14,4 +14,9 @@
   <xacro:property name="caster_radius"    value="0.025"/>
   <xacro:property name="body_rgba" value="${'0.20 0.47 0.96 1' if ns == 'robot1' else '0.94 0.55 0.16 1'}"/>
+  <xacro:arg name="cameras" default="true"/>
+  <xacro:arg name="camera_width" default="512"/>
+  <xacro:arg name="camera_height" default="288"/>
+  <xacro:arg name="camera_rate" default="8.0"/>
+  <xacro:property name="robot_visual" value="${'blue' if ns == 'robot1' else 'amber'}"/>
   <!-- ===== 2. Mass helpers (physics needs inertia for every moving part) ===== -->
   <xacro:macro name="box_inertia" params="m x y z">
@@ -33,6 +38,5 @@
   <link name="base_link">
     <visual>
-      <geometry><box size="${base_length} ${base_width} ${base_height}"/></geometry>
-      <material name="body_${ns}"><color rgba="${body_rgba}"/></material>
+      <geometry><mesh filename="package://factory_bot/models/robot_premium/meshes/body_${robot_visual}.obj"/></geometry>
     </visual>
     <collision>
@@ -50,7 +54,5 @@
     <link name="${prefix}_wheel_link">
       <visual>
-        <origin rpy="1.5707963 0 0"/>
-        <geometry><cylinder radius="${wheel_radius}" length="${wheel_width}"/></geometry>
-        <material name="wheel_black"><color rgba="0.1 0.1 0.1 1"/></material>
+        <geometry><mesh filename="package://factory_bot/models/robot_premium/meshes/wheel.obj"/></geometry>
       </visual>
        <collision>
@@ -103,7 +105,5 @@
     <!-- Housing drawn BELOW the sensor point: the lidar must not see its own case. -->
     <visual>
-      <origin xyz="0 0 -0.04"/>
-      <geometry><cylinder radius="0.035" length="0.03"/></geometry>
-      <material name="wheel_black"><color rgba="0.1 0.1 0.1 1"/></material>
+      <geometry><mesh filename="package://factory_bot/models/robot_premium/meshes/lidar.obj"/></geometry>
     </visual>
     <inertial>
@@ -116,4 +116,17 @@
     <child link="laser_link"/>
     <origin xyz="0.10 0 ${base_height/2 + 0.06}"/>
+  </joint>
+  <!-- Low front safety lidar: ahead of our own shell, at the other robot's body height.
+       The original 360-degree SLAM lidar and its reference-map scan plane stay unchanged. -->
+  <link name="obstacle_laser_link">
+    <visual>
+      <origin xyz="-0.015 0 0"/>
+      <geometry><box size="0.018 0.045 0.018"/></geometry>
+      <material name="safety_lidar_graphite"><color rgba="0.06 0.08 0.09 1"/></material>
+    </visual>
+  </link>
+  <joint name="obstacle_laser_joint" type="fixed">
+    <parent link="base_link"/><child link="obstacle_laser_link"/>
+    <origin xyz="0.205 0 0.010"/>
   </joint>
   <link name="imu_link">
@@ -128,4 +141,15 @@
     <origin xyz="0 0 0.02"/>
   </joint>
+  <!-- Visual camera lens is in the shell. Massless fixed sensor frames retain original dynamics. -->
+  <link name="camera_link"/>
+  <joint name="camera_joint" type="fixed">
+    <parent link="base_link"/><child link="camera_link"/>
+    <origin xyz="0.189 0 0.052"/>
+  </joint>
+  <link name="camera_optical_frame"/>
+  <joint name="camera_optical_joint" type="fixed">
+    <parent link="camera_link"/><child link="camera_optical_frame"/>
+    <origin rpy="-1.57079632679 0 -1.57079632679"/>
+  </joint>
   <xacro:include filename="$(find factory_bot)/urdf/fleet_bot.ros2_control.xacro"/>
   <xacro:include filename="$(find factory_bot)/urdf/fleet_bot.gazebo.xacro"/>

Commit message: Add dark pixel dashboard controls and bounded reverse recovery

File: src/factory_bot/urdf/fleet_bot.gazebo.xacro (robot description, xacro)
@@ -71,4 +71,20 @@
     </sensor>
   </gazebo>
+  <!-- Rear half-plane at body height: full-width reverse clearance, not mapping. -->
+  <gazebo reference="rear_obstacle_laser_link">
+    <sensor name="rear_obstacle_lidar_${ns}" type="gpu_lidar">
+      <topic>${ns}/rear_obstacle_scan</topic>
+      <gz_frame_id>${ns}/rear_obstacle_laser_link</gz_frame_id>
+      <update_rate>10</update_rate><always_on>true</always_on><visualize>false</visualize>
+      <lidar>
+        <visibility_mask>2415919103</visibility_mask>
+        <scan><horizontal><samples>181</samples><resolution>1</resolution>
+          <min_angle>-1.5707963267948966</min_angle><max_angle>1.5707963267948966</max_angle>
+        </horizontal></scan>
+        <range><min>0.02</min><max>4.0</max><resolution>0.01</resolution></range>
+        <noise><type>gaussian</type><mean>0.0</mean><stddev>0.005</stddev></noise>
+      </lidar>
+    </sensor>
+  </gazebo>
   <!-- First-person RGB camera. Sensor forward = +X; ROS optical frame = +Z forward. -->
   <xacro:if value="$(arg cameras)">

File: src/factory_bot/urdf/fleet_bot.urdf.xacro (robot description, xacro)
@@ -130,4 +130,16 @@
     <origin xyz="0.205 0 0.010"/>
   </joint>
+  <!-- Low rear safety lidar, outside our shell. It is not an ICP/SLAM input. -->
+  <link name="rear_obstacle_laser_link">
+    <visual>
+      <origin xyz="-0.015 0 0"/>
+      <geometry><box size="0.018 0.045 0.018"/></geometry>
+      <material name="safety_lidar_graphite"/>
+    </visual>
+  </link>
+  <joint name="rear_obstacle_laser_joint" type="fixed">
+    <parent link="base_link"/><child link="rear_obstacle_laser_link"/>
+    <origin xyz="-0.205 0 0.010" rpy="0 0 3.141592653589793"/>
+  </joint>
   <link name="imu_link">
     <inertial>
